File: DSM-Interfacer.kicad_sch (KiCad schematic)
At the start: 25 parts, among them J1 USB_B_Micro, J2 DIAG, Q1 BSS138, Q2 BSS138, Q3 MMBT2222A, SW1 RESET, SW2 BOOT/FLASH, U1 ESP32-WROOM-32, U2 MAX232, U3 CH340C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

Commit message: smaller MAX323
Parts:
- SW2: now left out of the parts list
- U2: footprint Package_DIP:DIP-16_W7.62mm -> Package_SO:SOIC-16_3.9x9.9mm_P1.27mm
Changed lines of the file:
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@@
       (effects (font (size 1.27 1.27)) (justify left))
     )
-    (property "Footprint" "Package_DIP:DIP-16_W7.62mm" (id 2) (at 177.8 106.68 0)
+    (property "Footprint" "Package_SO:SOIC-16_3.9x9.9mm_P1.27mm" (id 2) (at 177.8 106.68 0)
       (effects (font (size 1.27 1.27)) (justify left) hide)
     )
@@
   )
   (symbol (lib_id "Switch:SW_SPST") (at 90.805 102.235 0) (unit 1)
-    (in_bom yes) (on_board yes) (fields_autoplaced)
+    (in_bom no) (on_board no) (fields_autoplaced)
     (property "Reference" "SW2" (id 0) (at 90.805 96.6175 0))
     (property "Value" "BOOT/FLASH" (id 1) (at 90.805 99.3926 0))
@@
     )
     (path "/08aef537-b15e-4cd7-9de8-48074389e69b"
-      (reference "U2") (unit 1) (value "MAX232") (footprint "Package_DIP:DIP-16_W7.62mm")
+      (reference "U2") (unit 1) (value "MAX232") (footprint "Package_SO:SOIC-16_3.9x9.9mm_P1.27mm")
     )
     (path "/76a62690-f180-44fa-9ec9-7d6e6a9afe1f"
